File: MCU_Weather_Station.kicad_pcb (KiCad board)
At the start: 2 copper layers, 119.5 x 89.5 mm, 35 parts, among them J1 DC 5V Power, J2 USB_B, J3 AVR-ISP-6, SW1 MCU_RESET_BUTTON, SW2 SW_Push, U1 ATmega328-P, U2 Olimex_MOD-WIFI-ESP8266-DEV, U3 CH340C, U4 AMS1117-3.3, Y1 16MHz

Commit message: Add filled zones (GND front and bottom layer) and resolve all DRC errors
Parts:
- added REF**: KiCad-Logo2_5mm_SilkScreen, Symbol:KiCad-Logo2_5mm_SilkScreen, F.Cu at (149.5, 58.5)
Routing:
- net GND: track 411.5 -> 416.6 mm, vias 5 -> 7
- added copper zone on B.Cu, net GND
- added copper zone on F.Cu, net GND
Other:
- board text added: "READY"
- board text added: "WIFI"

Commit message: Add PCBWay directory for gerber and BOM files to manufacture
Other:
- board text added: "Designed by Alessio De Nicola Manufactured in China Version: 1.0"
- board text removed: "Designed by: Alessio De Nicola Manufactured in: Shenzen, China Version: 1.0"
Changed lines of the file:
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@@
 			(outputformat 1)
 			(mirror no)
-			(drillshape 1)
+			(drillshape 0)
 			(scaleselection 1)
-			(outputdirectory "")
+			(outputdirectory "PCBWay/")
 		)
 	)
@@
 		)
 	)
-	(gr_text "Designed by: Alessio De Nicola\nManufactured in: Shenzen, China\nVersion: 1.0"
+	(gr_text "Designed by Alessio De Nicola\nManufactured in China\nVersion: 1.0"
 		(at 86 50 0)
 		(layer "F.SilkS")
